File: KiCad project/ESP32-C3-02.kicad_sch (KiCad schematic)
At the start: 30 parts, among them J3 GSD090012SEU, U3 ESP32-C3-WROOM-02-H4, U4 CP2102N-A02-GQFN20, U5 USBLC6-2SC6, U6 W25Q32JVSSIQ

Commit message: added license and references
Other:
- company: Tech Explorations -> (none)
Changed lines of the file:
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@@
 	(title_block
 		(title "ESP32 C3 02 and USB to UART converter")
-		(date "2024-11-23")
+		(date "2026-01-24")
 		(rev "1")
-		(company "Tech Explorations")
 	)
 	(rectangle
