File: pcb/ESP32 sensor board.kicad_sch (KiCad schematic)
At the start: 26 parts, among them J1 USB_C_Receptacle, J2 JST_2mm_LiPo, U1 MCP73871, U2 LM1117MPX-3.3_NOPB

Commit message: created ibom document
Other:
- title: ESP32 sensor board -> (none)
