File: pcb/ESP32-C3-02.kicad_sch (KiCad schematic)
At the start: 30 parts, among them J3 GSD090012SEU, U3 ESP32-C3-WROOM-02-H4, U4 CP2102N-A02-GQFN20, U5 USBLC6-2SC6, U6 W25Q32JVSSIQ

Commit message: created ibom document
Other:
- title: ESP32 C3 02 and USB to UART converter -> (none)
