File: pcb/sensors.kicad_sch (KiCad schematic)
At the start: 23 parts, among them Q1 TEMT6000X01, U7 BME280, U8 MAX4466EXK+T

Commit message: created ibom document
Parts:
- U7: DESCRIPTION Integrated pressure, humidity and temperature sensor; 8-pin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 -> (none)
